Commit message: Update Gazebo simulation

File: gazebo_simulation/eufs_description/sensors/gps.urdf.xacro (robot description, xacro)
@@ -43,14 +43,14 @@
                 <frameId>${prefix}_base_link</frameId>
                 <topicName>/gps/fix</topicName>
-                <!-- Appleton Tower coordinates -->
-                <referenceLatitude>55.944400</referenceLatitude>
-                <referenceLongitude>-3.18629</referenceLongitude>
+                <!-- Garage coordinates -->
+                <referenceLatitude>59.35115</referenceLatitude>
+                <referenceLongitude>18.07042</referenceLongitude>
                 <!-- To set heading in ENU orientation (degrees) -->
                 <referenceHeading>0</referenceHeading>
                 <velocityTopicName>/gps/velocity</velocityTopicName>
                 <drift>0.0 0.0 0.0</drift>
-                <gaussianNoise>0.1 0.1 0.1</gaussianNoise>
+                <gaussianNoise>2.5 2.5 3.0</gaussianNoise>
                 <velocityDrift>0.00001 0.00001 0.00001</velocityDrift>
-                <velocityGaussianNoise>0.00001 0.00001 0.00001</velocityGaussianNoise>
+                <velocityGaussianNoise>0.05 0.05 0.05</velocityGaussianNoise>
             </plugin>
         </gazebo>

File: gazebo_simulation/eufs_description/sensors/imu.urdf.xacro (robot description, xacro)
@@ -31,9 +31,28 @@
 			<plugin filename="libgazebo_ros_imu.so" name="${prefix}_controller">
 				<alwaysOn>true</alwaysOn>
-				<bodyName>${prefix}_base_link</bodyName>
-				<topicName>${prefix}</topicName>
-				<serviceName>${prefix}_service</serviceName>
-				<gaussianNoise>0.005</gaussianNoise>
-				<updateRate>1000.0</updateRate>
+	      <bodyName>${prefix}_base_link</bodyName>
+	      <frameName>${prefix}_base_link</frameName>
+	      <topicName>${prefix}</topicName>
+	      <serviceName>${prefix}_service</serviceName>
+	      <gaussianNoise>0.01</gaussianNoise>
+	      <updateRate>100.0</updateRate>
+	      <imu>
+	        <noise>
+	          <type>gaussian</type>
+	          <rate>
+	            <mean>0.0</mean>
+	            <stddev>0.0</stddev>
+	            <stddev>2e-4</stddev>
+	            <bias_mean>0.0000075</bias_mean>
+	            <bias_stddev>0.0000008</bias_stddev>
+	          </rate>
+	          <accel>
+	            <mean>0.0</mean>
+	            <stddev>1.1e-2</stddev>
+	            <bias_mean>0.01</bias_mean>
+	            <bias_stddev>0.001</bias_stddev>
+	          </accel>
+	        </noise>
+	      </imu>
 			</plugin>
 		</gazebo>

File: gazebo_simulation/eufs_description/urdf/bases/ads-dv_base.urdf.xacro (robot description, xacro)
@@ -8,4 +8,6 @@
   <!-- <xacro:property name="clearance" value="${tire_dia/2.0}" /> -->
   <xacro:property name="clearance" value="0.25" />
+  <xacro:property name="offset_model" value="-0.85" />
+  <xacro:property name="height_model" value="-0.2" />
   <!-- BASE FOOTPRINT -->
   <xacro:if value="${publish_bf}">
@@ -37,23 +39,17 @@
       <mass value="125.0" />
       <origin xyz="0 0 0" />
+      <!-- TODO  -->
       <inertia  ixx="1.391" ixy="0.004"  ixz="0.0"  iyy="6.853"  iyz="0.0"  izz="6.125" />
     </inertial>
     <visual>
-       <origin xyz="0 0 0" rpy="0 0 0" />
-       <xacro:if value="${hq}">
+       <origin xyz="${offset_model} 0 ${height_model}" rpy="0 0 0" />
        <geometry>
-	     <mesh filename="package://eufs_description/meshes/ads-dv.dae"/>
+  	     <mesh filename="package://eufs_description/meshes/fs_car.dae"/>
        </geometry>
-       </xacro:if>
-       <xacro:unless value="${hq}">
-       <geometry>
-	     <mesh filename="package://eufs_description/meshes/ads-dv.dae"/>
-       </geometry>
-       </xacro:unless>
     </visual>
     <collision>
-       <origin xyz="0 0 0" rpy="0 0 0 " />
+       <origin xyz="${offset_model} 0 ${height_model}" rpy="0 0 0 " />
        <geometry>
-         <mesh filename="package://eufs_description/meshes/ads-dv.dae"/>
+         <mesh filename="package://eufs_description/meshes/fs_car.dae"/>
        </geometry>
     </collision>

File: gazebo_simulation/eufs_description/urdf/wheels/suspension_wheel.urdf.xacro (robot description, xacro)
@@ -15,6 +15,6 @@
        from a U joint to the corresponding hex hub. wheel_travel is the
        vertical wheel travel. -->
-  <xacro:property name="wheelbase" value="1.55"/>
-  <xacro:property name="hex_hub_dist" value="1.360"/>  <!-- track/width of the car -->
+  <xacro:property name="wheelbase" value="1.60"/>
+  <xacro:property name="hex_hub_dist" value="1.1"/>  <!-- track/width of the car -->
   <xacro:property name="axle_length" value="0.120"/>
   <xacro:property name="wheel_travel" value="0.05"/>
