Commit message: Increase IMU accuracy

File: gazebo_simulation/eufs_description/sensors/imu.urdf.xacro (robot description, xacro)
@@ -29,30 +29,21 @@
 		</link>
 		<gazebo>
-			<plugin filename="libgazebo_ros_imu.so" name="${prefix}_controller">
+			<plugin filename="libhector_gazebo_ros_imu.so" name="imu_plugin">
 				<alwaysOn>true</alwaysOn>
-	      <bodyName>${prefix}_base_link</bodyName>
-	      <frameName>${prefix}_base_link</frameName>
-	      <topicName>${prefix}</topicName>
-	      <serviceName>${prefix}_service</serviceName>
-	      <gaussianNoise>0.01</gaussianNoise>
-	      <updateRate>100.0</updateRate>
-	      <imu>
-	        <noise>
-	          <type>gaussian</type>
-	          <rate>
-	            <mean>0.0</mean>
-	            <stddev>0.0</stddev>
-	            <stddev>2e-4</stddev>
-	            <bias_mean>0.0000075</bias_mean>
-	            <bias_stddev>0.0000008</bias_stddev>
-	          </rate>
-	          <accel>
-	            <mean>0.0</mean>
-	            <stddev>1.1e-2</stddev>
-	            <bias_mean>0.01</bias_mean>
-	            <bias_stddev>0.001</bias_stddev>
-	          </accel>
-	        </noise>
-	      </imu>
+        <updateRate>100.0</updateRate>
+        <bodyName>${prefix}_base_link</bodyName>
+        <frameId>${prefix}_base_link</frameId>
+				<topicName>${prefix}</topicName>
+				<serviceName>${prefix}/calibrate</serviceName>
+        <rpyOffsets>0 0 0</rpyOffsets> 		<!-- deprecated -->
+        <gaussianNoise>0</gaussianNoise>  <!-- deprecated -->
+				<accelOffset>0.0 0.0 0.0</accelOffset>
+        <accelDrift>0.0 0.0 0.0</accelDrift>
+				<accelDriftFrequency>1.0 1.0 1.0</accelDriftFrequency>
+        <accelGaussianNoise>0.011 0.011 0.3</accelGaussianNoise>
+				<rateOffset>0.0 0.0 0.0</rateOffset>
+				<rateDrift>0.0 0.0 0.0</rateDrift>
+				<rateDriftFrequency>1.0 1.0 1.0</rateDriftFrequency>
+				<rateGaussianNoise>0.0 0.0 0.002</rateGaussianNoise>
 			</plugin>
 		</gazebo>

File: gazebo_simulation/eufs_description/urdf/wheels/suspension_wheel.urdf.xacro (robot description, xacro)
@@ -18,6 +18,8 @@
   <xacro:property name="hex_hub_dist" value="1.1"/>  <!-- track/width of the car -->
   <xacro:property name="axle_length" value="0.120"/>
-  <xacro:property name="wheel_travel" value="0.05"/>
-  <xacro:property name="shock_z_offset" value="0.05"/>
+  <xacro:property name="wheel_travel" value="0.0"/>
+  <!-- <xacro:property name="wheel_travel" value="0.05"/> -->
+  <xacro:property name="shock_z_offset" value="0.0"/>
+  <!-- <xacro:property name="shock_z_offset" value="0.05"/> -->
   <!-- Degree-to-radian conversions -->
   <xacro:property name="degrees_45" value="0.785398163"/>
@@ -25,6 +27,6 @@
   <xacro:property name="degrees_180" value="3.14159265"/>
   <!-- shock_eff_limit is 2 * ((shock_stroke / 2) * shock_spring_constant) N. -->
-  <xacro:property name="shock_eff_limit" value="50"/>
-  <xacro:property name="shock_vel_limit" value="500"/>
+  <xacro:property name="shock_eff_limit" value="500"/>
+  <xacro:property name="shock_vel_limit" value="5000"/>
   <xacro:property name="wheel_joint_damping" value="0.01" />
   <xacro:property name="wheel_joint_friction" value="0.1" />
